Commit message: Remove antenna model

File: urdf/leo.urdf.xacro (robot description, xacro)
@@ -4,5 +4,4 @@
   <xacro:arg name="robot_ns" default="leo"/>
   <xacro:arg name="fixed" default="false"/>
-  <xacro:arg name="default_antenna" default="true"/>
   <xacro:arg name="rockers_fixed" default="true"/>
   <xacro:include filename="$(find leo_description)/urdf/leo.gazebo.xacro"/>
@@ -94,27 +93,4 @@
   <xacro:wheel_link name="FR" model="B"/>
   <xacro:wheel_link name="RR" model="B"/>
-  <xacro:if value="$(arg default_antenna)">
-    <link name="antenna_link">
-      <inertial>
-        <mass value="0.001237"/>
-        <origin xyz="0 0 0.028828"/>
-        <inertia
-          ixx="2.5529e-7" ixy="0.0" ixz="0.0"
-          iyy="2.5529e-7" iyz="0.0"
-          izz="1.354e-8"/>
-      </inertial>
-      <visual>
-        <geometry>
-          <mesh filename="package://leo_description/models/Antenna.dae"/>
-        </geometry>
-      </visual>
-      <collision>
-        <origin xyz="0 0 0.028"/>
-        <geometry>
-          <cylinder radius="0.0055" length="0.056"/>
-        </geometry>
-      </collision>
-    </link>
-  </xacro:if>
   <link name="camera_frame"/>
   <link name="camera_optical_frame"/>
@@ -175,11 +151,4 @@
     <dynamics friction="0.3125" damping="0.1"/>
   </joint>
-  <xacro:if value="$(arg default_antenna)">
-    <joint name="antenna_joint" type="fixed">
-      <origin xyz="-0.0052 0.056 -0.0065" rpy="0 0 0"/>
-      <parent link="base_link"/>
-      <child link="antenna_link"/>
-    </joint>
-  </xacro:if>
   <joint name="camera_joint" type="fixed">
     <origin xyz="0.0971 0 -0.0427" rpy="0 0.2094 0"/>
