Commit message: Modify wheel friction parameters and collision models

File: urdf/include/leo.gazebo.xacro (robot description, xacro)
@@ -22,5 +22,5 @@
     <kp>1e6</kp>
     <kd>1.0</kd>
-    <mu1>5.0</mu1>
+    <mu1>3.0</mu1>
     <mu2>0.5</mu2>
     <fdir1>1 0 0</fdir1>
@@ -30,5 +30,5 @@
     <kp>1e6</kp>
     <kd>1.0</kd>
-    <mu1>5.0</mu1>
+    <mu1>3.0</mu1>
     <mu2>0.5</mu2>
     <fdir1>1 0 0</fdir1>
@@ -38,5 +38,5 @@
     <kp>1e6</kp>
     <kd>1.0</kd>
-    <mu1>5.0</mu1>
+    <mu1>3.0</mu1>
     <mu2>0.5</mu2>
     <fdir1>1 0 0</fdir1>
@@ -46,5 +46,5 @@
     <kp>1e6</kp>
     <kd>1.0</kd>
-    <mu1>5.0</mu1>
+    <mu1>3.0</mu1>
     <mu2>0.5</mu2>
     <fdir1>1 0 0</fdir1>

File: urdf/leo.urdf.xacro (robot description, xacro)
@@ -56,5 +56,11 @@
         <origin xyz="0 0.04485 0" rpy="${pi/2} 0 0"/>
         <geometry>
-          <cylinder radius="0.0625" length="0.07"/>
+          <cylinder radius="0.057" length="0.07"/>
+        </geometry>
+      </collision>
+      <collision>
+        <origin xyz="0 0.04485 0" rpy="${pi/2} 0 0"/>
+        <geometry>
+          <cylinder radius="0.0625" length="0.04"/>
         </geometry>
       </collision>
