Commit message: Update the ZED2 mast tilt angle

File: urdf/include/erc_setup.urdf.xacro (robot description, xacro)
@@ -28,5 +28,5 @@
   </link>
   <joint name="zed2_tilt_head_joint" type="fixed">
-    <origin xyz="0 0 0.1291" rpy="0 0.4 0"/>
+    <origin xyz="0 0 0.1291" rpy="0 0.415911961 0"/> <!-- 23.83 degree tilt -->
     <parent link="erc_setup_link"/>
     <child link="zed2_tilt_head_link"/>
